File: HoneyBee-V1.2.sch (EAGLE design)
At the start: 48 parts, among them IC2 CA3130EZLMP, Q1 2N5457

Commit message: Added SMD Fet layout
Added FET pads to layout. This is version 1.2
Parts:
- removed +9V: +9V(T), mb_supply:+9V(T)
- removed D6: 5v1 Zener, mb_diodes:1N9ZENER
- removed G1: GND(T), mb_supply:GND(T)
- removed IN1: IN(T), mb_supply:IN(T)
- removed L/SW: (no value), mb_supply:PAD
- removed LED: 3mm, mb_diodes:LED3MM
- removed OUT: OUT(T), mb_supply:OUT(T)
- removed R15: 1k, mb_resistors:6MM.3
- added U$1: MMBF5457, xc_library:MMBF5457
- added U$2: BOARDLINK, xc_library:BOARDLINK
- D4, D5: value 1N4007 -> 4007
- IC2: value CA3130EZLMP -> CA3130EZ
- renumbered NAT to TONE
Connections:
- removed net +9V: +9V.+9V, D5.A
- removed net IN: C1.1, IN1.IN, R1.2
- removed net OUT: OUT.OUT, VOL.2
- net GND: now also U$2.G; no longer G1.GND
- net N$16: now also U$1.G
- net N$17: now also U$1.S
- net N$18: now also U$1.D
- net N$20: now also C1.1, R1.2, U$2.IN; no longer LED.A, R15.2
- net N$23: no longer D6.C
- net N$24: now also D5.A, U$2.+9V; no longer D6.A, R15.1
- net N$25: now also U$2.OUT, VOL.2; no longer L/SW.PAD, LED.C
